File: KiCAD/MiniADSR 1.0/MiniADSR 1.0.kicad_pcb (KiCad board)
At the start: 2 copper layers, 105 x 128.5 mm, 50 parts, among them J1 INPUT, J2 OUTPUT, J3 JST_BUS, J4 ControlBoard_Pins, J5 IDC_BUS, J6 MainBoard_Pins, Q1 BC547, Q2 BC547, Q3 BC547, U1 LM555, U2 TL072

Commit message: Updated front panel labels
Routing:
- net Net-(C3-Pad1): track 40.6 -> 41.9 mm
- net GND2: vias 65 -> 68
- net (no net): vias 6 -> 4
Other:
- outline, holes or cut-outs redrawn
- board text added: "@benjiaomodular"
- board text added: "IN"
- board text added: "MiniADSR"
- board text added: "OUT"
