File: KiCAD/MiniADSR 1.1/Power.sch (KiCad schematic (older format))
At the start: 7 parts, among them J5 IDC_BUS, J7 JST_BUS, U2 TL072

Commit message: Redesigned PCB layout, added cap for longer decay
Parts:
- J7: footprint Connector_JST:JST_XH_B6B-XH-A_1x06_P2.50mm_Vertical -> Connector_JST:JST_XH_B3B-XH-A_1x03_P2.50mm_Vertical; symbol Connector:Conn_01x06_Male -> Connector:Conn_01x03_Male
Connections:
- net +12V: now also J7.1 (Pin_1); no longer J7.4 (Pin_4)
- net -12V: now also J7.3 (Pin_3); no longer J7.6 (Pin_6)
- net GND2: now also J7.2 (Pin_2); no longer J7.5 (Pin_5)
- no-connect marks 3 -> 0
Changed lines of the file:
@@
 $EndComp
 $Comp
-L Connector:Conn_01x06_Male J?
+L Connector:Conn_01x03_Male J?
 U 1 1 61FC4B84
-P 3950 3700
+P 3950 3900
 AR Path="/61FC4B84" Ref="J?"  Part="1"
 AR Path="/61FA9972/61FC4B84" Ref="J7"  Part="1"
 AR Path="/61F51CE9/61FC4B84" Ref="J5"  Part="1"
 AR Path="/61EBA3CC/61FC4B84" Ref="J3"  Part="1"
-F 0 "J3" H 4075 4200 50  0000 R CNN
-F 1 "JST_BUS" H 4200 4075 50  0000 R CNN
-F 2 "Connector_JST:JST_XH_B6B-XH-A_1x06_P2.50mm_Vertical" H 3950 3700 50  0001 C CNN
-F 3 "~" H 3950 3700 50  0001 C CNN
-	1    3950 3700
+F 0 "J3" H 4075 4400 50  0000 R CNN
+F 1 "JST_BUS" H 4200 4275 50  0000 R CNN
+F 2 "Connector_JST:JST_XH_B3B-XH-A_1x03_P2.50mm_Vertical" H 3950 3900 50  0001 C CNN
+F 3 "~" H 3950 3900 50  0001 C CNN
+	1    3950 3900
 	1    0    0    -1
 $EndComp
@@
 Wire Wire Line
 	4950 3975 4950 4050
-NoConn ~ 4150 3700
-NoConn ~ 4150 3600
-NoConn ~ 4150 3500
 $Comp
 L power:GND2 #PWR0104
